File: eagle/gps_tracker.brd (EAGLE design)
At the start: 99.1 x 29.3 mm, 57 parts, among them Q1 MC-405, U1 ORG1411, U2 ATMEGA328P_TQFP, U3 A2235-H, U4 AP7312

Commit message: Add files via upload
Parts:
- removed +1V8, +3V3_1, +3V3_2, +3V3_3, GND31, RXI, RXI1, TXO, VIN: (no value), wirepad:SMD1,27-2,54
- removed C15: (no value), rcl:C0603
- removed SJ1: ON, SparkFun-Passives:PAD-JUMPER-2-NC_BY_PASTE_YES_SILK
- added +VIN, +VIN2, +VIN_1, +VIN_2, ENA1, ENA2, ENA_1, ENA_2, RXI_1, RXI_2, TXO_: (no value), wirepad:SMD1,27-2,54
- added C18, C19, C20, C21: (no value), rcl:C0603
- added R10, R9: (no value), rcl:R0603
- added U$2: 1X2, headers(2mm)(samtec):1X2
- added U5, U6: ADP160, SparkFun-PowerIC:SOT23-5
- R6: device rcl:R1206 -> rcl:R0603
- U4: value AP7312 -> ADP160; device gps_tracker:SOT23-6 -> SparkFun-PowerIC:SOT23-5
- moved U4 36.9 mm to (73.0, 21.6), flipped to the bottom, turned to 90 degrees
- moved TXO2 30.5 mm to (67.3, 7.62), flipped to the bottom
- moved R3 21.7 mm to (109.9, 17.1), turned to 270 degrees
- moved LED2 21.3 mm to (89.5, 18.4), turned to 0 degrees
- moved R4 19.8 mm to (89.5, 15.2), turned to 90 degrees
- moved C6 14.1 mm to (106.7, 18.4), turned to 0 degrees
- moved C4 12.5 mm to (106.7, 17.1), turned to 0 degrees
- moved C5 11.1 mm to (106.7, 15.9), turned to 0 degrees
- moved LED1 8.28 mm to (75.6, 8.89), turned to 90 degrees
- moved R1 6.25 mm to (62.9, 10.2)
- moved TXO1 5.75 mm to (99.7, 8.26), turned to 90 degrees
- moved C2 5.43 mm to (74.3, 18.4), turned to 0 degrees
- moved R6 3.42 mm to (39.4, 24.1), turned to 90 degrees
- moved C3 3.24 mm to (74.3, 17.1), turned to 0 degrees
- moved R2 2.62 mm to (76.8, 11.4), turned to 270 degrees
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- renumbered GND to GND40
Connections:
- removed net N$11: RXI.1, RXI1.1, U2.30
- removed net N$18: C14.1, SJ1.1, U4.3, U4.4
- new net ENA: ENA_1.1, ENA_2.1, R6.2, U6.3
- new net N$23: ENA1.1, R9.2, U5.3
- new net N$25: ENA2.1, R10.2, U4.3
- new net N$27: C4.1, C5.1, C6.1, R3.2, U3.3, U5.5
- new net RXI: RXI_1.1, RXI_2.1, U2.30
- net +3V3: now also U6.5; no longer +3V3_1.1, +3V3_2.1, +3V3_3.1, C4.1, C5.1, C6.1, R3.2, R6.1, U3.3, U4.1
- net +4.1V: now also +VIN.1, +VIN2.1, +VIN_1.1, +VIN_2.1, C14.1, C18.1, C19.1, C20.1, C21.1, R10.1, R6.1, R9.1, U$2.1, U4.1, U5.1, U6.1; no longer SJ1.2, U4.5, VIN.1
- net GND: now also C18.2, C19.2, C20.2, C21.2, U$2.2, U5.2, U6.2; no longer C15.2, GND31.1
- net N$17: now also TXO_.1; no longer TXO2.1
- net N$5: now also TXO2.1; no longer TXO.1
- net V+: now also U4.5; no longer +1V8.1, C15.1, R6.2, U4.6
Routing:
- net +3V3: track 88.1 -> 48.0 mm, vias 4 -> 1
- net +4.1V: track 5.95 -> 30.1 mm, vias 0 -> 1
- net N$27: track 0.00 -> 18.9 mm, vias 0 -> 1
- net RXI: track 0.00 -> 18.4 mm, vias 0 -> 1
- net N$11: track 13.5 -> 0.00 mm, vias 1 -> 0
- net N$5: track 8.95 -> 20.3 mm
- net N$9: track 33.9 -> 24.1 mm
- net ENA: track 0.00 -> 8.62 mm, vias 0 -> 1
- net V+: track 18.0 -> 25.7 mm
- net GND: track 19.9 -> 12.3 mm, vias 9 -> 10
- net N$18: track 7.33 -> 0.00 mm
- net N$23: track 0.00 -> 5.90 mm
- net N$25: track 0.00 -> 4.63 mm
- net N$10: track 16.2 -> 12.1 mm
- net N$2: track 6.45 -> 9.26 mm
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Other:
- board size 99.1 x 29.3 mm -> 99.7 x 29.3 mm

Commit message: Add files via upload
Parts:
- removed BUZ+, BUZ-: (no value), wirepad:SMD1,27-2,54
- added C15: (no value), rcl:C0603
- added LED3: (no value), led:CHIPLED_0603
- added R11, R12, R13: (no value), rcl:R0603
- added U$3, U$4: 1X2, headers(2mm)(samtec):1X2
- added U7: MCP73831, SparkFun-PowerIC:SOT23-5
- moved R8 4.84 mm to (20.3, 21.0), turned to 270 degrees
- moved R7 3.86 mm to (20.3, 23.5)
- moved Q2 3.81 mm to (18.4, 23.5)
- moved C12 3.18 mm to (24.1, 24.1)
- moved C13 3.18 mm to (27.3, 24.1)
- moved Q1 1.91 mm to (25.4, 21.6)
- moved +VIN2 0.64 mm to (67.3, 19.7)
- moved +VIN_1 0.64 mm to (45.7, 21.0)
- moved +VIN_2 0.64 mm to (45.7, 21.0)
- moved GND17 0.64 mm to (45.7, 18.4)
- moved GND24 0.64 mm to (45.7, 18.4)
- moved GND40 0.64 mm to (67.3, 17.1)
- moved R10 0.64 mm to (69.8, 21.0)
- moved U$2 0.64 mm to (39.4, 22.2)
- moved U4 0.64 mm to (73.0, 21.0)
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Connections:
- new net N$11: R12.1, U7.5
- new net N$18: LED3.C, U7.1
- new net N$22: LED3.A, R13.2
- new net N$24: C15.1, R13.1, U$4.1, U7.4
- net !CS: now also R11.2
- net +3V3: now also R11.1, U$3.2, U2.11
- net +4.1V: now also U7.3; no longer BUZ+.1
- net GND: now also C15.2, R12.2, U$4.2, U7.2
- net N$21: now also U$3.1; no longer BUZ-.1
Routing:
- net +3V3: track 48.0 -> 64.6 mm
- net +4.1V: track 30.1 -> 43.3 mm
- net N$24: track 0.00 -> 12.9 mm, vias 0 -> 1
- net GND: track 12.3 -> 20.4 mm
- net N$20: track 3.34 -> 8.20 mm
- net N$19: track 4.02 -> 1.79 mm
- net N$11: track 0.00 -> 1.92 mm
- net N$18: track 0.00 -> 1.82 mm
- net RF_RTTY: track 19.9 -> 18.6 mm
- net N$22: track 0.00 -> 0.94 mm
- net RXI: track 18.4 -> 17.5 mm
- net N$21: track 1.70 -> 0.80 mm
- net N$16: track 5.56 -> 6.38 mm
- net N$15: track 8.75 -> 9.46 mm
Other:
- outline, holes or cut-outs redrawn

Commit message: Add files via upload
Parts:
- added C22: 100nF, rcl:C0603
- added C23: (no value), rcl:C1206
- added C24, C25, C26: (no value), rcl:C0603
- added C27: 0.22uF, rcl:C0603K
- added C28: 0.22uF, rcl:C0603
- added IC1: MS563702BA03, freetronics-original:MS5637
- added JP1: (no value), pinhead:2X03
- added LED4, LED6: (no value), led:CHIPLED_0805
- added Q3, Q4: 200mA/50V, SparkFun-DiscreteSemi:SOT23-3
- added Q5: (no value), SparkFun-DiscreteSemi:SOT23-3
- added R14, R15, R18, R19, R20, R24, R25, R27: (no value), rcl:R0603
- added R16, R17: (no value), rcl:R1206
- added R21, R30: 220, resistor:R0603
- added RXIH: (no value), wirepad:SMD1,27-2,54
- added TP1, TP3: TPSB1,27, testpad:B1,27
- added U$5, U$6, U$7, U$8: 1X2, headers(2mm)(samtec):1X2
- added U11: ADP160, SparkFun-PowerIC:SOT23-5
- added U8: Tiny45-20-SMT, SparkFun-DigitalIC:SO08-EIAJ
- added U9: LIS3MDL, kg-ic:VFLGA-12
- moved LED2 26.0 mm to (64.8, 10.5), turned to 90 degrees
- moved R1 13.2 mm to (50.8, 15.6), turned to 270 degrees
- moved LED1 11.6 mm to (78.7, 20.0), turned to 0 degrees
- moved C20 10.9 mm to (60.3, 18.1)
- moved C21 10.9 mm to (60.3, 19.4)
- moved C4 10.9 mm to (95.9, 18.7)
- moved C5 10.9 mm to (95.9, 17.5)
- moved C6 10.9 mm to (95.9, 20.0)
- moved R3 10.9 mm to (99.1, 18.7)
- moved U4 10.9 mm to (62.2, 22.5)
- moved U5 10.9 mm to (95.9, 23.2)
- moved !RES 10.9 mm to (29.2, 14.3)
- moved +VIN2 10.9 mm to (56.5, 21.3)
- moved +VIN_1 10.9 mm to (34.9, 22.5)
- moved +VIN_2 10.9 mm to (34.9, 22.5)
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Connections:
- new net BUZZER: R30.2, TP3.TP, U8.6
- new net N$26: Q3.3, R16.1, TXO2.1
- new net N$28: Q5.3, U$7.1
- new net N$29: C24.1, R20.2, TP1.TP, U8.1
- new net N$30: Q4.3, R17.1, RXIH.1
- new net N$31: Q5.1, R18.2, R19.2, U$8.2
- new net N$32: Q4.2, R14.1, U1.10
- new net N$33: LED4.A, R21.1
- new net N$34: R27.2, U11.3
- new net N$35: LED6.A, R30.1
- new net N$36: C27.2, U9.4
- new net PYRO: R18.1, R21.2, U8.2
- new net SCL: IC1.3, R25.2, U8.7, U9.1
- new net SDA: IC1.2, R24.2, U8.5, U9.11
- new net UART: U$6.2, U8.3
- new net VBAT: C25.1, R27.1, U$5.1, U$7.2, U11.1
- new net VCC: C22.1, C23.1, C26.1, C28.1, IC1.1, R20.1, R24.1, R25.1, U11.5, U8.8, U9.10, U9.5, U9.6, U9.9
- net +4.1V: now also R16.2, R17.2
- net GND: now also C22.2, C23.2, C24.2, C25.2, C26.2, C27.1, C28.2, IC1.4, JP1.1, JP1.3, JP1.5, LED4.C, LED6.C, Q5.2, R19.1, U$5.2, U$6.1, U$8.1, U11.2, U8.4, U9.12, U9.2, U9.3
- net N$4: now also LED2.A; no longer LED1.A
- net N$5: now also Q3.2, R15.2; no longer TXO2.1
- net N$7: now also LED1.A; no longer LED2.A
- net V+: now also Q3.1, Q4.1, R14.2, R15.1
Routing:
- net VCC: track 0.00 -> 38.3 mm, vias 0 -> 2
- net +4.1V: track 43.3 -> 68.0 mm
- net SDA: track 0.00 -> 18.0 mm, vias 0 -> 1
- net SCL: track 0.00 -> 16.6 mm, vias 0 -> 1
- net PYRO: track 0.00 -> 12.5 mm
- net V+: track 25.4 -> 35.5 mm
- net VBAT: track 0.00 -> 8.59 mm
- net N$5: track 20.3 -> 12.8 mm
- net UART: track 0.00 -> 7.46 mm
- net N$26: track 0.00 -> 6.53 mm
- net GND: track 20.4 -> 27.0 mm, vias 10 -> 17
- net N$29: track 0.00 -> 6.27 mm
- net N$32: track 0.00 -> 5.87 mm, vias 0 -> 1
- net N$1: track 34.5 -> 39.4 mm
- net N$2: track 9.26 -> 4.67 mm
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Other:
- board size 99.7 x 29.3 mm -> 101 x 64.2 mm

Commit message: Add files via upload
Parts:
- removed JP1: (no value), pinhead:2X03
- added C29: (no value), rcl:C0603
- added LED5: (no value), led:CHIPLED_0603
- added R22, R23: (no value), rcl:R0603
- added U$9: 1X2, headers(2mm)(samtec):1X2
- added U10: MCP73831, SparkFun-PowerIC:SOT23-5
Connections:
- new net N$37: R22.1, U10.5
- new net N$38: LED5.C, U10.1
- new net N$39: LED5.A, R23.2
- new net N$40: C29.1, R23.1, U$9.1, U10.4
- net GND: now also C29.2, R22.2, U$9.2, U10.2; no longer JP1.1, JP1.3, JP1.5
- net VBAT: now also U10.3
Routing:
- net N$40: track 0.00 -> 11.3 mm
- net VBAT: track 8.59 -> 15.8 mm, vias 0 -> 1
- net N$37: track 0.00 -> 2.18 mm
- net N$39: track 0.00 -> 1.84 mm
- net N$38: track 0.00 -> 1.63 mm
- net VCC: track 38.3 -> 39.0 mm
- net GND: vias 17 -> 18
Other:
- board size 101 x 64.2 mm -> 99.7 x 64.2 mm
