File: eagle/gps_tracker.sch (EAGLE design)
At the start: 57 parts, among them Q1 MC-405, Q2 MOSFET-NCHANNELAO3404A, U1 ORG1411, U2 ATMEGA328P_TQFP, U3 A2235-H, U4 AP7312

Commit message: Add files via upload
Parts:
- removed +1V8, +3V3_1, +3V3_2, +3V3_3, GND, GND31, RXI, RXI1, TXO, VIN: (no value), wirepad:SMD2
- removed C15: (no value), rcl:C-EUC0603
- removed SJ1: ON, SparkFun-Passives:JUMPER-PAD-2-NC_BY_PASTE
- added +VIN, +VIN2, +VIN_1, +VIN_2, ENA1, ENA2, ENA_1, ENA_2, GND40, RXI_1, RXI_2, TXO_: (no value), wirepad:SMD2
- added C18, C19, C20, C21: (no value), rcl:C-EUC0603
- added R10, R9: (no value), rcl:R-EU_R0603
- added U$2: 1X2, headers(2mm)(samtec):1X2
- added U5, U6: ADP160, SparkFun-PowerIC:ADP160
- R6: device rcl:R-EU_R1206 -> rcl:R-EU_R0603
- U4: value AP7312 -> ADP160; device gps_tracker:AP7312 -> SparkFun-PowerIC:ADP160; FARNELL 2138328 -> 2510505
Connections:
- removed net N$11: RXI.P, RXI1.P, U2.PD0(RXD)
- removed net N$18: C14.1, SJ1.1, U4.EN1, U4.EN2
- new net ENA: ENA_1.P, ENA_2.P, R6.2, U6.EN
- new net N$23: ENA1.P, R9.2, U5.EN
- new net N$25: ENA2.P, R10.2, U4.EN
- new net N$27: C4.1, C5.1, C6.1, R3.2, U3.+3V3, U5.VOUT
- new net RXI: RXI_1.P, RXI_2.P, U2.PD0(RXD)
- net +3V3: now also U6.VOUT; no longer +3V3_1.P, +3V3_2.P, +3V3_3.P, C4.1, C5.1, C6.1, R3.2, R6.1, U3.+3V3, U4.3V3
- net +4.1V: now also +VIN.P, +VIN2.P, +VIN_1.P, +VIN_2.P, C14.1, C18.1, C19.1, C20.1, C21.1, R10.1, R6.1, R9.1, U$2.1, U4.VIN, U5.VIN, U6.VIN; no longer SJ1.2, U4.IN, VIN.P
- net GND: now also C18.2, C19.2, C20.2, C21.2, GND40.P, U$2.2, U5.GND, U6.GND; no longer C15.2, GND.P, GND31.P
- net N$17: now also TXO_.P; no longer TXO2.P
- net N$5: now also TXO2.P; no longer TXO.P
- net V+: now also U4.VOUT; no longer +1V8.P, C15.1, R6.2, U4.1V8
Other:
- moved on the sheet: C1, C14, C2, C3, C4, C5, C6, GND15, GND17, GND24, LED1, LED2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

Commit message: Add files via upload
Parts:
- removed BUZ+, BUZ-: (no value), wirepad:SMD2
- added C15: (no value), rcl:C-EUC0603
- added LED3: (no value), led:LEDCHIPLED_0603
- added R11, R12, R13: (no value), rcl:R-EU_R0603
- added U$3, U$4: 1X2, headers(2mm)(samtec):1X2
- added U7: MCP73831, SparkFun-PowerIC:MCP73831
Connections:
- new net N$11: R12.1, U7.PROG
- new net N$18: LED3.C, U7.STAT
- new net N$22: LED3.A, R13.2
- new net N$24: C15.1, R13.1, U$4.1, U7.VIN
- net !CS: now also R11.2
- net +3V3: now also R11.1, U$3.2, U2.PD7(AIN1)
- net +4.1V: now also U7.VBAT; no longer BUZ+.P
- net GND: now also C15.2, R12.2, U$4.2, U7.VSS
- net N$21: now also U$3.1; no longer BUZ-.P

Commit message: Add files via upload
Parts:
- added C22: 100nF, rcl:C-EUC0603
- added C23: (no value), rcl:C-EUC1206
- added C24, C25, C26: (no value), rcl:C-EUC0603
- added C27: 0.22uF, rcl:C-EUC0603K
- added C28: 0.22uF, rcl:C-EUC0603
- added IC1: MS563702BA03, freetronics-original:MS563702BA03
- added JP1: (no value), pinhead:PINHD-2X3
- added LED4, LED6: (no value), led:LEDCHIPLED_0805
- added Q3, Q4: 200mA/50V, SparkFun-DiscreteSemi:MOSFET-NCHANNELBSS138
- added Q5: MOSFET-NCHANNELBSS123LT1G, SparkFun-DiscreteSemi:MOSFET-NCHANNELBSS123LT1G
- added R14, R15, R18, R19, R20, R24, R25, R27: (no value), rcl:R-EU_R0603
- added R16, R17: (no value), rcl:R-EU_R1206
- added R21, R30: 220, resistor:R-EU_R0603
- added RXIH: (no value), wirepad:SMD2
- added TP1, TP3: TPSB1,27, testpad:TPSB1,27
- added U$5, U$6, U$7, U$8: 1X2, headers(2mm)(samtec):1X2
- added U11: ADP160, SparkFun-PowerIC:ADP160
- added U8: Tiny45-20-SMT, SparkFun-DigitalIC:ATTINY45TINY45-20-SMT
- added U9: LIS3MDL, kg-ic:LIS3MDL
Connections:
- new net BUZZER: R30.2, TP3.PP, U8.PB1(MISO)
- new net N$26: Q3.D, R16.1, TXO2.P
- new net N$28: Q5.D, U$7.1
- new net N$29: C24.1, R20.2, TP1.PP, U8.PB5(NRES)
- new net N$30: Q4.D, R17.1, RXIH.P
- new net N$31: Q5.G, R18.2, R19.2, U$8.2
- new net N$32: Q4.S, R14.1, U1.RXI/MOSI/SDA
- new net N$33: LED4.A, R21.1
- new net N$34: R27.2, U11.EN
- new net N$35: LED6.A, R30.1
- new net N$36: C27.2, U9.C1
- new net PYRO: R18.1, R21.2, U8.PB3(ADC3)
- new net SCL: IC1.SCL, R25.2, U8.PB2(SCK/ADC1), U9.SCL/SPC
- new net SDA: IC1.SDA, R24.2, U8.PB0(MOSI), U9.SDA/SDI
- new net UART: U$6.2, U8.PB4(ADC2)
- new net VBAT: C25.1, R27.1, U$5.1, U$7.2, U11.VIN
- new net VCC: C22.1, C23.1, C26.1, C28.1, IC1.VDD, R20.1, R24.1, R25.1, U11.VOUT, U8.VCC, U9.CS, U9.SD0/SA1, U9.VDD, U9.VDD_IO
- net +4.1V: now also R16.2, R17.2
- net GND: now also C22.2, C23.2, C24.2, C25.2, C26.2, C27.1, C28.2, IC1.GND, JP1.1, JP1.3, JP1.5, LED4.C, LED6.C, Q5.S, R19.1, U$5.2, U$6.1, U$8.1, U11.GND, U8.GND, U9.GND, U9.RSVD1, U9.RSVD2
- net N$4: now also LED2.A; no longer LED1.A
- net N$5: now also Q3.S, R15.2; no longer TXO2.P
- net N$7: now also LED1.A; no longer LED2.A
- net V+: now also Q3.G, Q4.G, R14.2, R15.1

Commit message: Add files via upload
Parts:
- removed JP1: (no value), pinhead:PINHD-2X3
- added C29: (no value), rcl:C-EUC0603
- added LED5: (no value), led:LEDCHIPLED_0603
- added R22, R23: (no value), rcl:R-EU_R0603
- added U$9: 1X2, headers(2mm)(samtec):1X2
- added U10: MCP73831, SparkFun-PowerIC:MCP73831
Connections:
- new net N$37: R22.1, U10.PROG
- new net N$38: LED5.C, U10.STAT
- new net N$39: LED5.A, R23.2
- new net N$40: C29.1, R23.1, U$9.1, U10.VIN
- net GND: now also C29.2, R22.2, U$9.2, U10.VSS; no longer JP1.1, JP1.3, JP1.5
- net VBAT: now also U10.VBAT
Other:
- moved on the sheet: C25, C26, R27, U$5, U11
