File: eagle/flight.sch (EAGLE design)
At the start: 142 parts, among them IC2 MS563702BA03, Q1 MC-405, Q10 MOSFET-NCHANNELBSS123LT1G, Q13 MC-405, Q14 MOSFET-NCHANNELAO3404A, Q2 MOSFET-NCHANNELAO3404A, Q7 200mA/50V, Q8 200mA/50V, U10 ORG1411, U13 ADP160, U19 Tiny45-20-SMT, U2 ATMEGA328P_TQFP, U20 LIS3MDL, U21 ADP160, U22 MCP73831, U3 A2235-H, U34 ATMEGA328P_TQFP, U37 ADP160, U38 MCP73831, U5 ADP160, U6 ADP160, U7 MCP73831

Commit message: Add files via upload
Parts:
- removed !RES, !RES3, ANT, ANT2, MISO, MISO3, MOSI, MOSI3, RXI1, RXIH, RXI_1, RXI_5, SCK, SCK3, TXO1, TXO4, TXO_, TXO_3: (no value), wirepad:SMD2
- removed C10, C101, C11, C12, C13, C14, C15, C16, C17, C18, C19, C22, C23, C24, C4, C40, C41, C5, C6, C7, C8, C89, C9, C90, C91, C92, C93, C94, C95, C96, C97, C98: (no value), rcl:C-EUC0603
- removed LED1, LED21, LED3, LED4: (no value), led:LEDCHIPLED_0603
- removed Q13: MC-405, gps_tracker:MC-405
- removed Q14: MOSFET-NCHANNELAO3404A, SparkFun-DiscreteSemi:MOSFET-NCHANNELAO3404A
- removed Q7, Q8: 200mA/50V, SparkFun-DiscreteSemi:MOSFET-NCHANNELBSS138
- removed R10, R11, R12, R13, R14, R22, R23, R31, R35, R36, R4, R5, R6, R7, R8, R88, R89, R9, R90, R92, R93, R94, R95: (no value), rcl:R-EU_R0603
- removed R37, R38: (no value), rcl:R-EU_R1206
- removed U$1, U$35: RFM69HW, hoperf:RFM69HW
- removed U$2, U$3, U$36, U$37, U$38, U$39, U$4, U$9: 1X2, headers(2mm)(samtec):1X2
- removed U10: ORG1411, gps_tracker:ORG1411
- removed U13, U37, U5, U6: ADP160, SparkFun-PowerIC:ADP160
- removed U2, U34: ATMEGA328P_TQFP, SparkFun-DigitalIC:ATMEGA328P_TQFP
- removed U3: A2235-H, gps_tracker:A2235-H
- removed U38, U7: MCP73831, SparkFun-PowerIC:MCP73831
- added CAM, CAM_ENA, ENA: 1X2, headers(2mm)(samtec):1X2
- Q1: value MC-405 -> MOSFET-PCHANNEL; device gps_tracker:MC-405 -> SparkFun-DiscreteSemi:MOSFET-PCHANNEL; FARNELL 2508596 -> (none)
- Q2: value MOSFET-NCHANNELAO3404A -> MOSFET-NCHANNELBSS123LT1G; device SparkFun-DiscreteSemi:MOSFET-NCHANNELAO3404A -> SparkFun-DiscreteSemi:MOSFET-NCHANNELBSS123LT1G
- R1, R2, R3: value (none) -> 220; device rcl:R-EU_R0603 -> resistor:R-EU_R0603
- renumbered U$14 to BAT, U$15 to UART, U$16 to PYRO, U$18 to CHAR
Connections:
- removed net !CS1: R11.2, U$1.NSS, U2.PB1(OC1A)
- removed net !CS2: R93.2, U$35.NSS, U34.PB1(OC1A)
- removed net !RF_RES1: U$1.RESET, U2.PD2(INT0)
- removed net !RF_RES2: U$35.RESET, U34.PD2(INT0)
- removed net +3V3_1: C10.1, C11.1, C16.1, C17.1, C9.1, R11.1, R5.2, U$1.VCC, U$3.2, U2.AVCC, U2.PC3(ADC3), U2.PD7(AIN1), U2.VCC@4, U2.VCC@6, U6.VOUT
- removed net +3V3_2: C91.1, C92.1, C93.1, C97.1, C98.1, R88.2, R93.1, U$35.VCC, U$37.2, U34.AVCC, U34.PC3(ADC3), U34.PD7(AIN1), U34.VCC@4, U34.VCC@6, U37.VOUT
- removed net +4.1V: R37.2, R38.2
- removed net +BAT1: C14.1, R2.2, R6.1, U$2.1, U6.VIN, U7.VBAT
- removed net +BAT2: C40.1, C41.1, C96.1, R31.1, R92.1, U$36.1, U13.VIN, U37.VIN, U38.VBAT
- removed net ANT2: ANT2.P, U$35.ANT
- removed net ENA1: R1.2, R6.2, U$9.2, U6.EN
- removed net ENA2: R31.2, R92.2, U$39.2, U13.EN, U37.EN
- removed net GND1: C10.2, C11.2, C12.2, C13.2, C14.2, C15.2, C16.2, C17.2, C18.2, C19.2, C4.2, C5.2, C6.2, C7.2, C8.2, C9.2, LED1.C, Q2.S, R12.2, R7.1, U$1.GNDA, U$1.GNDB, U$2.2, U$4.2, U$9.1, U2.AGND, U2.GND@3, U2.GND@5, U3.EXTINT, U3.GND6, U3.GND9, U5.GND, U6.GND, U7.VSS
- removed net GND2: C101.2, C22.2, C23.2, C24.2, C40.2, C41.2, C89.2, C90.2, C91.2, C92.2, C93.2, C94.2, C95.2, C96.2, C97.2, C98.2, LED4.C, Q14.S, R89.1, R94.2, U$35.GNDA, U$35.GNDB, U$36.2, U$38.2, U$39.1, U10.GND, U13.GND, U34.AGND, U34.GND@3, U34.GND@5, U37.GND, U38.VSS
- removed net MISO1: MISO.P, U$1.MISO, U2.PB4(MISO)
- removed net MISO2: MISO3.P, U$35.MISO, U34.PB4(MISO)
- removed net MOSI1: MOSI.P, U$1.MOSI, U2.PB3(MOSI/OC2)
- removed net MOSI2: MOSI3.P, U$35.MOSI, U34.PB3(MOSI/OC2)
- removed net N$11: R12.1, U7.PROG
- removed net N$12: C7.1, U2.AREF
- removed net N$13: !RES.P, C8.1, R5.1, U2.PC6(/RESET)
- removed net N$136: R51.2, U21.EN
- removed net N$14: ANT.P, U$1.ANT
- removed net N$15: C12.1, Q1.2, U2.PB7(XTAL2/TOSC2)
- removed net N$16: C13.1, Q1.1, U2.PB6(XTAL1/TOSC1)
- removed net N$162: C89.1, U34.AREF
- removed net N$163: !RES3.P, C90.1, R88.1, U34.PC6(/RESET)
- removed net N$165: C94.1, Q13.2, U34.PB7(XTAL2/TOSC2)
- removed net N$166: C95.1, Q13.1, U34.PB6(XTAL1/TOSC1)
- removed net N$167: Q14.G, R89.2, R90.1
- removed net N$168: R90.2, U34.PD6(AIN0)
- removed net N$169: Q14.D, U$37.1
- removed net N$171: R94.1, U38.PROG
- removed net N$172: LED21.C, U38.STAT
- removed net N$173: LED21.A, R95.2
- removed net N$174: C101.1, R95.1, U$38.1, U38.VIN
- removed net N$18: LED3.C, U7.STAT
- removed net N$19: Q2.G, R7.2, R8.1
- removed net N$20: R8.2, U2.PD6(AIN0)
- removed net N$21: Q2.D, U$3.1
- removed net N$22: LED3.A, R13.2
- removed net N$24: C15.1, R13.1, U$4.1, U7.VIN
- removed net N$27: C4.1, C5.1, C6.1, R3.2, U3.+3V3, U5.VOUT
- removed net N$29: U10.ON/OFF, U10.WAKEUP
- removed net N$30: R22.1, U10.MODE1/SCK/!CTS
- removed net N$31: R23.1, U10.1PPS
- removed net N$32: LED4.A, R23.2
- removed net N$54: Q7.S, R36.2, U10.TXO/MISO/SCL
- removed net N$55: Q7.D, R37.1, TXO4.P
- removed net N$56: Q8.D, R38.1, RXIH.P
- removed net N$57: Q8.S, R35.1, U10.RXI/MOSI/SDA
- removed net N$6: R3.1, U3.GPIO6
- removed net N$7: LED1.A, R4.2
- removed net N$8: R4.1, U3.TM_GPIO5
- removed net N$9: U3.ON_OFF, U3.WAKEUP
- removed net RF_RTTY1: U$1.DIO2, U2.PC1(ADC1)
- removed net RF_RTTY2: U$35.DIO2, U34.PC1(ADC1)
- removed net RXI1: R14.2, RXI_1.P, U2.PD0(RXD)
- removed net RXI2: RXI_5.P, U34.PD0(RXD)
- removed net RXI_G1: R10.1, RXI1.P, U3.RXI
- removed net SCK1: SCK.P, U$1.SCK, U2.PB5(SCK)
- removed net SCK2: SCK3.P, U$35.SCK, U34.PB5(SCK)
- removed net TXO1: R10.2, TXO_.P, U2.PD1(TXD)
- removed net TXO2: TXO_3.P, U34.PD1(TXD)
- removed net TXO_G1: R14.1, TXO1.P, U3.TXO
- removed net V+: C22.1, C23.1, C24.1, Q7.G, Q8.G, R22.2, R35.2, R36.1, U10.+1V8, U13.VOUT
- new net ENA: ENA.2, R51.2, U21.EN
- new net N$1: Q2.D, R2.2
- new net N$4: CAM_ENA.1, Q2.G, R3.1
- net GND: now also CAM.1, CAM_ENA.2, ENA.1, Q2.S
- net N$2: now also CAM.2, Q1.D; no longer R1.1, R9.2, U5.EN
- net N$3: now also Q1.G, R1.2; no longer C18.1, C19.1, R9.1, U5.VIN
- net VBAT: now also Q1.S, R1.1, R3.2
