File: eagle/gps_tracker_mark3.brd (EAGLE design)
At the start: 87.9 x 69.9 mm, 142 parts, among them IC2 MS563702BA03, Q1 MC-405, Q13 MC-405, Q7 200mA/50V, Q8 200mA/50V, U10 ORG1411, U13 ADP160, U19 Tiny45-20-SMT, U2 ATMEGA328P_TQFP, U20 LIS3MDL, U21 ADP160, U22 MCP73831, U3 A2235-H, U34 ATMEGA328P_TQFP, U37 ADP160, U38 MCP73831, U5 ADP160, U6 ADP160, U7 MCP73831

Commit message: Add files via upload
Parts:
- removed !RES3, ANT2, MISO3, MOSI3, RXIH, RXI_5, SCK3, TXO4, TXO_3: (no value), wirepad:SMD1,27-2,54
- removed C101, C22, C23, C24, C40, C41, C89, C90, C91, C92, C93, C94, C95, C96, C97, C98: (no value), rcl:C0603
- removed LED21, LED4: (no value), led:CHIPLED_0603
- removed Q13: MC-405, gps_tracker:MC-405
- removed Q14: (no value), SparkFun-DiscreteSemi:SOT23-3
- removed Q7, Q8: 200mA/50V, SparkFun-DiscreteSemi:SOT23-3
- removed R22, R23, R31, R35, R36, R88, R89, R90, R92, R93, R94, R95: (no value), rcl:R0603
- removed R37, R38: (no value), rcl:R1206
- removed U$35: RFM69HW, hoperf:RFM
- removed U$36, U$37, U$38, U$39: 1X2, headers(2mm)(samtec):1X2
- removed U10: ORG1411, gps_tracker:ORG1411
- removed U13, U37: ADP160, SparkFun-PowerIC:SOT23-5
- removed U34: ATMEGA328P_TQFP, SparkFun-DigitalIC:TQFP32-08
- removed U38: MCP73831, SparkFun-PowerIC:SOT23-5
Connections:
- removed net !CS2: R93.2, U$35.NSS, U34.13
- removed net !RF_RES2: U$35.RESET, U34.32
- removed net +3V3_2: C91.1, C92.1, C93.1, C97.1, C98.1, R88.2, R93.1, U$35.VCC, U$37.2, U34.11, U34.18, U34.26, U34.4, U34.6, U37.5
- removed net +4.1V: R37.2, R38.2
- removed net +BAT2: C40.1, C41.1, C96.1, R31.1, R92.1, U$36.1, U13.1, U37.1, U38.3
- removed net ANT2: ANT2.1, U$35.ANT
- removed net ENA2: R31.2, R92.2, U$39.2, U13.3, U37.3
- removed net GND2: C101.2, C22.2, C23.2, C24.2, C40.2, C41.2, C89.2, C90.2, C91.2, C92.2, C93.2, C94.2, C95.2, C96.2, C97.2, C98.2, LED4.C, Q14.2, R89.1, R94.2, U$35.GNDA, U$35.GNDB, U$36.2, U$38.2, U$39.1, U10.11, U10.5, U13.2, U34.21, U34.3, U34.5, U37.2, U38.2
- removed net MISO2: MISO3.1, U$35.MISO, U34.16
- removed net MOSI2: MOSI3.1, U$35.MOSI, U34.15
- removed net N$162: C89.1, U34.20
- removed net N$163: !RES3.1, C90.1, R88.1, U34.29
- removed net N$165: C94.1, Q13.2, U34.8
- removed net N$166: C95.1, Q13.1, U34.7
- removed net N$167: Q14.1, R89.2, R90.1
- removed net N$168: R90.2, U34.10
- removed net N$169: Q14.3, U$37.1
- removed net N$171: R94.1, U38.5
- removed net N$172: LED21.C, U38.1
- removed net N$173: LED21.A, R95.2
- removed net N$174: C101.1, R95.1, U$38.1, U38.4
- removed net N$29: U10.1, U10.6
- removed net N$30: R22.1, U10.7
- removed net N$31: R23.1, U10.2
- removed net N$32: LED4.A, R23.2
- removed net N$54: Q7.2, R36.2, U10.3
- removed net N$55: Q7.3, R37.1, TXO4.1
- removed net N$56: Q8.3, R38.1, RXIH.1
- removed net N$57: Q8.2, R35.1, U10.10
- removed net RF_RTTY2: U$35.DIO2, U34.24
- removed net RXI2: RXI_5.1, U34.30
- removed net SCK2: SCK3.1, U$35.SCK, U34.17
- removed net TXO2: TXO_3.1, U34.31
- removed net V+: C22.1, C23.1, C24.1, Q7.1, Q8.1, R22.2, R35.2, R36.1, U10.4, U13.5
Routing:
- net N$29: track 39.4 -> 0.00 mm, vias 2 -> 0
- net VCC: track 0.00 -> 39.1 mm, vias 0 -> 2
- net V+: track 35.5 -> 0.00 mm, vias 1 -> 0
- net GND1: track 69.4 -> 38.9 mm, vias 19 -> 10
- net +4.1V: track 22.8 -> 0.00 mm
- net RF_RTTY1: track 0.00 -> 21.6 mm, vias 0 -> 1
- net SDA: track 0.00 -> 18.0 mm, vias 0 -> 1
- net SCL: track 0.00 -> 16.6 mm, vias 0 -> 1
- net VBAT: track 0.00 -> 15.8 mm, vias 0 -> 1
- net !CS1: track 0.00 -> 13.0 mm, vias 0 -> 1
- net N$174: track 12.9 -> 0.00 mm, vias 1 -> 0
- net N$54: track 12.8 -> 0.00 mm, vias 1 -> 0
- net RXI1: track 0.00 -> 12.6 mm
- net PYRO: track 0.00 -> 12.5 mm
- net RXI2: track 12.2 -> 0.00 mm
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- removed copper zone on layer 1, net GND2
- removed copper zone on layer 16, net GND2
Other:
- board size 87.9 x 69.9 mm -> 87.9 x 28 mm
