File: eagle/gps_tracker_mark3.sch (EAGLE design)
At the start: 142 parts, among them IC2 MS563702BA03, Q1 MC-405, Q10 MOSFET-NCHANNELBSS123LT1G, Q13 MC-405, Q14 MOSFET-NCHANNELAO3404A, Q2 MOSFET-NCHANNELAO3404A, Q7 200mA/50V, Q8 200mA/50V, U10 ORG1411, U13 ADP160, U19 Tiny45-20-SMT, U2 ATMEGA328P_TQFP, U20 LIS3MDL, U21 ADP160, U22 MCP73831, U3 A2235-H, U34 ATMEGA328P_TQFP, U37 ADP160, U38 MCP73831, U5 ADP160, U6 ADP160, U7 MCP73831

Commit message: Add files via upload
Parts:
- removed !RES3, ANT2, MISO3, MOSI3, RXIH, RXI_5, SCK3, TXO4, TXO_3: (no value), wirepad:SMD2
- removed C101, C22, C23, C24, C40, C41, C89, C90, C91, C92, C93, C94, C95, C96, C97, C98: (no value), rcl:C-EUC0603
- removed LED21, LED4: (no value), led:LEDCHIPLED_0603
- removed Q13: MC-405, gps_tracker:MC-405
- removed Q14: MOSFET-NCHANNELAO3404A, SparkFun-DiscreteSemi:MOSFET-NCHANNELAO3404A
- removed Q7, Q8: 200mA/50V, SparkFun-DiscreteSemi:MOSFET-NCHANNELBSS138
- removed R22, R23, R31, R35, R36, R88, R89, R90, R92, R93, R94, R95: (no value), rcl:R-EU_R0603
- removed R37, R38: (no value), rcl:R-EU_R1206
- removed U$35: RFM69HW, hoperf:RFM69HW
- removed U$36, U$37, U$38, U$39: 1X2, headers(2mm)(samtec):1X2
- removed U10: ORG1411, gps_tracker:ORG1411
- removed U13, U37: ADP160, SparkFun-PowerIC:ADP160
- removed U34: ATMEGA328P_TQFP, SparkFun-DigitalIC:ATMEGA328P_TQFP
- removed U38: MCP73831, SparkFun-PowerIC:MCP73831
Connections:
- removed net !CS2: R93.2, U$35.NSS, U34.PB1(OC1A)
- removed net !RF_RES2: U$35.RESET, U34.PD2(INT0)
- removed net +3V3_2: C91.1, C92.1, C93.1, C97.1, C98.1, R88.2, R93.1, U$35.VCC, U$37.2, U34.AVCC, U34.PC3(ADC3), U34.PD7(AIN1), U34.VCC@4, U34.VCC@6, U37.VOUT
- removed net +4.1V: R37.2, R38.2
- removed net +BAT2: C40.1, C41.1, C96.1, R31.1, R92.1, U$36.1, U13.VIN, U37.VIN, U38.VBAT
- removed net ANT2: ANT2.P, U$35.ANT
- removed net ENA2: R31.2, R92.2, U$39.2, U13.EN, U37.EN
- removed net GND2: C101.2, C22.2, C23.2, C24.2, C40.2, C41.2, C89.2, C90.2, C91.2, C92.2, C93.2, C94.2, C95.2, C96.2, C97.2, C98.2, LED4.C, Q14.S, R89.1, R94.2, U$35.GNDA, U$35.GNDB, U$36.2, U$38.2, U$39.1, U10.GND, U13.GND, U34.AGND, U34.GND@3, U34.GND@5, U37.GND, U38.VSS
- removed net MISO2: MISO3.P, U$35.MISO, U34.PB4(MISO)
- removed net MOSI2: MOSI3.P, U$35.MOSI, U34.PB3(MOSI/OC2)
- removed net N$162: C89.1, U34.AREF
- removed net N$163: !RES3.P, C90.1, R88.1, U34.PC6(/RESET)
- removed net N$165: C94.1, Q13.2, U34.PB7(XTAL2/TOSC2)
- removed net N$166: C95.1, Q13.1, U34.PB6(XTAL1/TOSC1)
- removed net N$167: Q14.G, R89.2, R90.1
- removed net N$168: R90.2, U34.PD6(AIN0)
- removed net N$169: Q14.D, U$37.1
- removed net N$171: R94.1, U38.PROG
- removed net N$172: LED21.C, U38.STAT
- removed net N$173: LED21.A, R95.2
- removed net N$174: C101.1, R95.1, U$38.1, U38.VIN
- removed net N$29: U10.ON/OFF, U10.WAKEUP
- removed net N$30: R22.1, U10.MODE1/SCK/!CTS
- removed net N$31: R23.1, U10.1PPS
- removed net N$32: LED4.A, R23.2
- removed net N$54: Q7.S, R36.2, U10.TXO/MISO/SCL
- removed net N$55: Q7.D, R37.1, TXO4.P
- removed net N$56: Q8.D, R38.1, RXIH.P
- removed net N$57: Q8.S, R35.1, U10.RXI/MOSI/SDA
- removed net RF_RTTY2: U$35.DIO2, U34.PC1(ADC1)
- removed net RXI2: RXI_5.P, U34.PD0(RXD)
- removed net SCK2: SCK3.P, U$35.SCK, U34.PB5(SCK)
- removed net TXO2: TXO_3.P, U34.PD1(TXD)
- removed net V+: C22.1, C23.1, C24.1, Q7.G, Q8.G, R22.2, R35.2, R36.1, U10.+1V8, U13.VOUT
