File: eagle/flight.brd (EAGLE design)
At the start: 23 x 28 mm, 42 parts, among them IC2 MS563702BA03, Q1 MOSFET-PCHANNEL, U19 Tiny45-20-SMT, U20 LIS3MDL, U21 ADP160, U22 MCP73831

Commit message: Add files via upload
Parts:
- moved C53 0.37 mm to (3.47, 9.45)
Routing:
- added copper zone on layer 1, net N$5
- added copper zone on layer 16, net N$6
Changed lines of the file:
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@@
 <setting verticaltext="up"/>
 </settings>
-<grid distance="0.635" unitdist="mm" unit="mm" style="lines" multiple="1" display="yes" altdistance="0.025" altunitdist="inch" altunit="mm"/>
+<grid distance="0.3715" unitdist="mm" unit="mm" style="lines" multiple="1" display="yes" altdistance="0.025" altunitdist="inch" altunit="mm"/>
 <layers>
 <layer number="1" name="Top" color="4" fill="1" visible="yes" active="yes"/>
@@
 <element name="C51" library="rcl" package="C0603" value="100nF" x="9.520321875" y="17.809103125" rot="MR0"/>
 <element name="C52" library="rcl" package="C1206" value="" x="11.76285" y="7.234159375" rot="R270"/>
-<element name="C53" library="rcl" package="C0603" value="" x="3.837490625" y="9.4518625" rot="R90"/>
+<element name="C53" library="rcl" package="C0603" value="" x="3.465990625" y="9.4518625" rot="R90"/>
 <element name="C54" library="rcl" package="C0603" value="" x="14.465740625" y="17.839034375" rot="R90"/>
 <element name="IC2" library="freetronics-original" package="MS5637" value="MS563702BA03" x="9.520321875" y="15.269103125" rot="MR0"/>
@@
 <contactref element="CAM_ENA" pad="2"/>
 <wire x1="3.175" y1="14.605" x2="2.54" y2="15.875" width="0.5" layer="1"/>
-<wire x1="3.837490625" y1="10.3018625" x2="3.837490625" y2="10.767509375" width="0.5" layer="1"/>
+<wire x1="3.465990625" y1="10.3018625" x2="3.837490625" y2="10.767509375" width="0.5" layer="1"/>
 <wire x1="3.837490625" y1="10.767509375" x2="3.175" y2="11.43" width="0.5" layer="1"/>
 <wire x1="14.283690625" y1="5.42993125" x2="14.27913125" y2="5.42405" width="0" layer="19" extent="1-1"/>
@@
 <contactref element="C53" pad="1"/>
 <contactref element="TP2" pad="TP"/>
-<wire x1="3.837490625" y1="8.6018625" x2="4.940321875" y2="8.6018625" width="0.5" layer="1"/>
+<wire x1="3.465990625" y1="8.6018625" x2="4.940321875" y2="8.6018625" width="0.5" layer="1"/>
 <wire x1="4.940321875" y1="8.6018625" x2="4.940321875" y2="8.769103125" width="0.5" layer="1"/>
 <wire x1="6.345321875" y1="4.905903125" x2="6.345321875" y2="5.304103125" width="0.5" layer="1"/>
@@
 <wire x1="3.595" y1="12.53" x2="4.13" y2="13.065" width="0.5" layer="16"/>
 </signal>
+<signal name="N$5">
+<polygon width="0.01" layer="1" isolate="0.01">
+<vertex x="0.635" y="23.495"/>
+<vertex x="3.81" y="23.495"/>
+<vertex x="3.81" y="20.955"/>
+<vertex x="0.635" y="20.955"/>
+</polygon>
+</signal>
+<signal name="N$6">
+<polygon width="0.01" layer="16" isolate="0.01">
+<vertex x="0.635" y="20.955"/>
+<vertex x="3.81" y="20.955"/>
+<vertex x="3.81" y="23.495"/>
+<vertex x="0.635" y="23.495"/>
+</polygon>
+</signal>
 </signals>
