File: eagle/gps_tracker_A2235h.sch (EAGLE design)
At the start: 142 parts, among them IC2 MS563702BA03, Q1 MC-405, Q10 MOSFET-NCHANNELBSS123LT1G, Q13 MC-405, Q14 MOSFET-NCHANNELAO3404A, Q2 MOSFET-NCHANNELAO3404A, Q7 200mA/50V, Q8 200mA/50V, U10 ORG1411, U13 ADP160, U19 Tiny45-20-SMT, U2 ATMEGA328P_TQFP, U20 LIS3MDL, U21 ADP160, U22 MCP73831, U3 A2235-H, U34 ATMEGA328P_TQFP, U37 ADP160, U38 MCP73831, U5 ADP160, U6 ADP160, U7 MCP73831

Commit message: Add files via upload
Parts:
- removed !RES3, ANT2, MISO3, MOSI3, RXIH, RXI_5, SCK3, TXO4, TXO_3: (no value), wirepad:SMD2
- removed C101, C22, C23, C24, C40, C41, C53, C54, C55, C58, C89, C90, C91, C92, C93, C94, C95, C96, C97, C98: (no value), rcl:C-EUC0603
- removed C51: 100nF, rcl:C-EUC0603
- removed C52: (no value), rcl:C-EUC1206
- removed C56: 0.22uF, rcl:C-EUC0603K
- removed C57: 0.22uF, rcl:C-EUC0603
- removed IC2: MS563702BA03, freetronics-original:MS563702BA03
- removed LED10, LED11: (no value), led:LEDCHIPLED_0805
- removed LED12, LED21, LED4: (no value), led:LEDCHIPLED_0603
- removed Q10: MOSFET-NCHANNELBSS123LT1G, SparkFun-DiscreteSemi:MOSFET-NCHANNELBSS123LT1G
- removed Q13: MC-405, gps_tracker:MC-405
- removed Q14: MOSFET-NCHANNELAO3404A, SparkFun-DiscreteSemi:MOSFET-NCHANNELAO3404A
- removed Q7, Q8: 200mA/50V, SparkFun-DiscreteSemi:MOSFET-NCHANNELBSS138
- removed R22, R23, R31, R35, R36, R45, R46, R47, R49, R50, R51, R53, R54, R88, R89, R90, R92, R93, R94, R95: (no value), rcl:R-EU_R0603
- removed R37, R38: (no value), rcl:R-EU_R1206
- removed R48, R52: 220, resistor:R-EU_R0603
- removed TP2, TP4: TPSB1,27, testpad:TPSB1,27
- removed U$14, U$15, U$16, U$17, U$18, U$36, U$37, U$38, U$39: 1X2, headers(2mm)(samtec):1X2
- removed U$35: RFM69HW, hoperf:RFM69HW
- removed U10: ORG1411, gps_tracker:ORG1411
- removed U13, U21, U37: ADP160, SparkFun-PowerIC:ADP160
- removed U19: Tiny45-20-SMT, SparkFun-DigitalIC:ATTINY45TINY45-20-SMT
- removed U20: LIS3MDL, kg-ic:LIS3MDL
- removed U22, U38: MCP73831, SparkFun-PowerIC:MCP73831
- removed U34: ATMEGA328P_TQFP, SparkFun-DigitalIC:ATMEGA328P_TQFP
Connections:
- removed net !CS2: R93.2, U$35.NSS, U34.PB1(OC1A)
- removed net !RF_RES2: U$35.RESET, U34.PD2(INT0)
- removed net +3V3_2: C91.1, C92.1, C93.1, C97.1, C98.1, R88.2, R93.1, U$35.VCC, U$37.2, U34.AVCC, U34.PC3(ADC3), U34.PD7(AIN1), U34.VCC@4, U34.VCC@6, U37.VOUT
- removed net +4.1V: R37.2, R38.2
- removed net +BAT2: C40.1, C41.1, C96.1, R31.1, R92.1, U$36.1, U13.VIN, U37.VIN, U38.VBAT
- removed net ANT2: ANT2.P, U$35.ANT
- removed net BUZZER: R52.2, TP4.PP, U19.PB1(MISO)
- removed net ENA2: R31.2, R92.2, U$39.2, U13.EN, U37.EN
- removed net GND: C51.2, C52.2, C53.2, C54.2, C55.2, C56.1, C57.2, C58.2, IC2.GND, LED10.C, LED11.C, Q10.S, R46.1, R53.2, U$14.2, U$15.1, U$17.1, U$18.2, U19.GND, U20.GND, U20.RSVD1, U20.RSVD2, U21.GND, U22.VSS
- removed net GND2: C101.2, C22.2, C23.2, C24.2, C40.2, C41.2, C89.2, C90.2, C91.2, C92.2, C93.2, C94.2, C95.2, C96.2, C97.2, C98.2, LED4.C, Q14.S, R89.1, R94.2, U$35.GNDA, U$35.GNDB, U$36.2, U$38.2, U$39.1, U10.GND, U13.GND, U34.AGND, U34.GND@3, U34.GND@5, U37.GND, U38.VSS
- removed net MISO2: MISO3.P, U$35.MISO, U34.PB4(MISO)
- removed net MOSI2: MOSI3.P, U$35.MOSI, U34.PB3(MOSI/OC2)
- removed net N$132: C53.1, R47.2, TP2.PP, U19.PB5(NRES)
- removed net N$133: Q10.G, R45.2, R46.2, U$17.2
- removed net N$134: LED10.A, R48.1
- removed net N$135: C56.2, U20.C1
- removed net N$136: R51.2, U21.EN
- removed net N$137: LED11.A, R52.1
- removed net N$138: Q10.D, U$16.1
- removed net N$139: R53.1, U22.PROG
- removed net N$140: LED12.C, U22.STAT
- removed net N$141: LED12.A, R54.2
- removed net N$142: C58.1, R54.1, U$18.1, U22.VIN
- removed net N$162: C89.1, U34.AREF
- removed net N$163: !RES3.P, C90.1, R88.1, U34.PC6(/RESET)
- removed net N$165: C94.1, Q13.2, U34.PB7(XTAL2/TOSC2)
- removed net N$166: C95.1, Q13.1, U34.PB6(XTAL1/TOSC1)
- removed net N$167: Q14.G, R89.2, R90.1
- removed net N$168: R90.2, U34.PD6(AIN0)
- removed net N$169: Q14.D, U$37.1
- removed net N$171: R94.1, U38.PROG
- removed net N$172: LED21.C, U38.STAT
- removed net N$173: LED21.A, R95.2
- removed net N$174: C101.1, R95.1, U$38.1, U38.VIN
- removed net N$29: U10.ON/OFF, U10.WAKEUP
- removed net N$30: R22.1, U10.MODE1/SCK/!CTS
- removed net N$31: R23.1, U10.1PPS
- removed net N$32: LED4.A, R23.2
- removed net N$54: Q7.S, R36.2, U10.TXO/MISO/SCL
- removed net N$55: Q7.D, R37.1, TXO4.P
- removed net N$56: Q8.D, R38.1, RXIH.P
- removed net N$57: Q8.S, R35.1, U10.RXI/MOSI/SDA
- removed net PYRO: R45.1, R48.2, U19.PB3(ADC3)
- removed net RF_RTTY2: U$35.DIO2, U34.PC1(ADC1)
- removed net RXI2: RXI_5.P, U34.PD0(RXD)
- removed net SCK2: SCK3.P, U$35.SCK, U34.PB5(SCK)
- removed net SCL: IC2.SCL, R50.2, U19.PB2(SCK/ADC1), U20.SCL/SPC
- removed net SDA: IC2.SDA, R49.2, U19.PB0(MOSI), U20.SDA/SDI
- removed net TXO2: TXO_3.P, U34.PD1(TXD)
- removed net UART: U$15.2, U19.PB4(ADC2)
- removed net V+: C22.1, C23.1, C24.1, Q7.G, Q8.G, R22.2, R35.2, R36.1, U10.+1V8, U13.VOUT
- removed net VBAT: C54.1, R51.1, U$14.1, U$16.2, U21.VIN, U22.VBAT
- removed net VCC: C51.1, C52.1, C55.1, C57.1, IC2.VDD, R47.1, R49.1, R50.1, U19.VCC, U20.CS, U20.SD0/SA1, U20.VDD, U20.VDD_IO, U21.VOUT

Commit message: Add files via upload
Parts:
- removed U$1: RFM69HW, hoperf:RFM69HW
- added U$5: RFM69HW, gps_tracker:RFM69HW
Connections:
- net !CS1: now also U$5.NSS; no longer U$1.NSS
- net !RF_RES1: now also U$5.RESET; no longer U$1.RESET
- net +3V3_1: now also U$5.VCC; no longer U$1.VCC
- net GND1: now also U$5.GNDA, U$5.GNDB; no longer U$1.GNDA, U$1.GNDB
- net MISO1: now also U$5.MISO; no longer U$1.MISO
- net MOSI1: now also U$5.MOSI; no longer U$1.MOSI
- net N$14: now also U$5.ANT; no longer U$1.ANT
- net RF_RTTY1: now also U$5.DIO2; no longer U$1.DIO2
- net SCK1: now also U$5.SCK; no longer U$1.SCK
Changed lines of the file:
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@@
 <part name="GND2" library="supply1" deviceset="GND" device=""/>
 <part name="+3V2" library="supply1" deviceset="+3V3" device=""/>
-<part name="U$1" library="hoperf" deviceset="RFM69HW" device=""/>
 <part name="GND4" library="supply1" deviceset="GND" device=""/>
 <part name="R3" library="rcl" deviceset="R-EU_" device="R0603"/>
@@
 <part name="R10" library="rcl" deviceset="R-EU_" device="R0603"/>
 <part name="R14" library="rcl" deviceset="R-EU_" device="R0603"/>
+<part name="U$5" library="gps_tracker" deviceset="RFM69HW" device=""/>
 </parts>
 <sheets>
@@
 <instance part="GND2" gate="1" x="78.74" y="91.44"/>
 <instance part="+3V2" gate="G$1" x="33.02" y="91.44" rot="R180"/>
-<instance part="U$1" gate="A" x="55.88" y="116.84"/>
 <instance part="GND4" gate="1" x="0" y="0"/>
 <instance part="R3" gate="G$1" x="220.98" y="121.92" rot="R90"/>
@@
 <instance part="R10" gate="G$1" x="284.48" y="157.48"/>
 <instance part="R14" gate="G$1" x="284.48" y="137.16"/>
+<instance part="U$5" gate="A" x="55.88" y="116.84"/>
 </instances>
 <busses>
@@
 <wire x1="78.74" y1="109.22" x2="78.74" y2="99.06" width="0.1524" layer="91"/>
 <junction x="78.74" y="99.06"/>
-<pinref part="U$1" gate="A" pin="GNDB"/>
-<pinref part="U$1" gate="A" pin="GNDA"/>
+<pinref part="U$5" gate="A" pin="GNDB"/>
+<pinref part="U$5" gate="A" pin="GNDA"/>
 </segment>
 <segment>
@@
 <wire x1="36.83" y1="99.06" x2="33.02" y2="99.06" width="0.1524" layer="91"/>
 <wire x1="33.02" y1="99.06" x2="33.02" y2="93.98" width="0.1524" layer="91"/>
-<pinref part="U$1" gate="A" pin="VCC"/>
+<pinref part="U$5" gate="A" pin="VCC"/>
 </segment>
 <segment>
@@
 <wire x1="78.74" y1="114.3" x2="74.93" y2="114.3" width="0.1524" layer="91"/>
 <label x="78.74" y="114.3" size="1.778" layer="95" xref="yes"/>
-<pinref part="U$1" gate="A" pin="SCK"/>
+<pinref part="U$5" gate="A" pin="SCK"/>
 </segment>
 </net>
@@
 <wire x1="78.74" y1="119.38" x2="74.93" y2="119.38" width="0.1524" layer="91"/>
 <label x="78.74" y="119.38" size="1.778" layer="95" xref="yes"/>
-<pinref part="U$1" gate="A" pin="MISO"/>
+<pinref part="U$5" gate="A" pin="MISO"/>
 </segment>
 </net>
@@
 <wire x1="78.74" y1="124.46" x2="74.93" y2="124.46" width="0.1524" layer="91"/>
 <label x="78.74" y="124.46" size="1.778" layer="95" xref="yes"/>
-<pinref part="U$1" gate="A" pin="MOSI"/>
+<pinref part="U$5" gate="A" pin="MOSI"/>
 </segment>
 </net>
@@
 <segment>
 <label x="78.74" y="129.54" size="1.778" layer="95" xref="yes"/>
-<pinref part="U$1" gate="A" pin="NSS"/>
 <wire x1="74.93" y1="129.54" x2="78.74" y2="129.54" width="0.1524" layer="91"/>
+<pinref part="U$5" gate="A" pin="NSS"/>
 </segment>
 <segment>
@@
 <pinref part="ANT" gate="1" pin="P"/>
 <wire x1="83.82" y1="104.14" x2="74.93" y2="104.14" width="0.1524" layer="91"/>
-<pinref part="U$1" gate="A" pin="ANT"/>
+<pinref part="U$5" gate="A" pin="ANT"/>
 </segment>
 </net>
@@
 <segment>
 <label x="33.02" y="134.62" size="1.778" layer="95" rot="R180" xref="yes"/>
-<pinref part="U$1" gate="A" pin="RESET"/>
 <wire x1="36.83" y1="134.62" x2="33.02" y2="134.62" width="0.1524" layer="91"/>
+<pinref part="U$5" gate="A" pin="RESET"/>
 </segment>
 <segment>
@@
 <segment>
 <label x="33.02" y="119.38" size="1.778" layer="95" rot="R180" xref="yes"/>
-<pinref part="U$1" gate="A" pin="DIO2"/>
 <wire x1="36.83" y1="119.38" x2="33.02" y2="119.38" width="0.1524" layer="91"/>
-</segment>
-<segment>
+<pinref part="U$5" gate="A" pin="DIO2"/>
+</segment>
+<segment>
