File: eagle/flight-mag3110.sch (EAGLE design)
At the start: 54 parts, among them Q1 MC-405, Q2 MOSFET-NCHANNELAO3404A, U2 ATMEGA328P_TQFP, U3 A2235-H, U5 ADP160, U6 ADP160, U7 MCP73831

Commit message: Add files via upload
Parts:
- removed !RES, ANT, MISO, MOSI, RXI1, RXI_1, SCK, TXO1, TXO_: (no value), wirepad:SMD2
- removed C10, C17, C19, C5, C7, C8: 100n, rcl:C-EUC0603
- removed C11, C6: 1n, rcl:C-EUC0603
- removed C12, C13: 22p, rcl:C-EUC0603
- removed C14, C15, C16, C18, C9: 10uF, rcl:C-EUC0603
- removed LED1, LED3: (no value), led:LEDCHIPLED_0603
- removed Q1: MC-405, gps_tracker:MC-405
- removed Q2: MOSFET-NCHANNELAO3404A, SparkFun-DiscreteSemi:MOSFET-NCHANNELAO3404A
- removed R1, R10, R14, R2: 0, rcl:R-EU_R0603
- removed R11, R15, R3, R5: 10k, rcl:R-EU_R0603
- removed R12: 2k7, rcl:R-EU_R0603
- removed R13: 470, rcl:R-EU_R0603
- removed R4, R8: 220, rcl:R-EU_R0603
- removed R6, R7, R9: 100k, rcl:R-EU_R0603
- removed U$2, U$3, U$4, U$9: 1X2, headers(2mm)(samtec):1X2
- removed U$5: RFM69HW, gps_tracker:RFM69HW
- removed U2: ATMEGA328P_TQFP, SparkFun-DigitalIC:ATMEGA328P_TQFP
- removed U3: A2235-H, gps_tracker:A2235-H
- removed U5, U6: ADP160, SparkFun-PowerIC:ADP160
- removed U7: MCP73831, SparkFun-PowerIC:MCP73831
- added BAT, CHAR, ENA, PYRO, U$17, UART: 1X2, headers(2mm)(samtec):1X2
- added C1, C2, C3, C51, C53: 100n, rcl:C-EUC0603
- added C52: 100n, rcl:C-EUC1206
- added C54, C55, C58: 10uF, rcl:C-EUC0603
- added IC2: MS563702BA03, freetronics-original:MS563702BA03
- added LED10, LED11: (no value), led:LEDCHIPLED_0805
- added LED12: (no value), led:LEDCHIPLED_0603
- added Q10: MOSFET-NCHANNELBSS123LT1G, SparkFun-DiscreteSemi:MOSFET-NCHANNELBSS123LT1G
- added R45, R46: (no value), rcl:R-EU_R0603
- added R47: 10k, rcl:R-EU_R0603
- added R48, R52: 220, resistor:R-EU_R0603
- added R49, R50: 2k2, rcl:R-EU_R0603
- added R51: 100k, rcl:R-EU_R0603
- added R53: 5k6, rcl:R-EU_R0603
- added R54: 470, rcl:R-EU_R0603
- added TP2, TP4: TPSB1,27, testpad:TPSB1,27
- added U1: MAG3110FCR1, gps_tracker:MAG3110FCR1
- added U19: Tiny45-20-SMT, SparkFun-DigitalIC:ATTINY45TINY45-20-SMT
- added U21: ADP160, SparkFun-PowerIC:ADP160
- added U22: MCP73831, SparkFun-PowerIC:MCP73831
- C4: value 10uF -> 100n
Connections:
- removed net !CS1: R11.2, U$5.NSS, U2.PB1(OC1A)
- removed net !RF_RES1: U$5.RESET, U2.PD2(INT0)
- removed net +3V3_1: C10.1, C11.1, C16.1, C17.1, C9.1, R11.1, R15.2, R5.2, U$3.2, U$5.VCC, U2.AVCC, U2.PC3(ADC3), U2.PD7(AIN1), U2.VCC@4, U2.VCC@6, U6.VOUT
- removed net +BAT1: C14.1, R2.2, R6.1, U$2.1, U6.VIN, U7.VBAT
- removed net ENA1: R1.2, R6.2, U$9.2, U6.EN
- removed net GND1: C10.2, C11.2, C12.2, C13.2, C14.2, C15.2, C16.2, C17.2, C18.2, C19.2, C4.2, C5.2, C6.2, C7.2, C8.2, C9.2, LED1.C, Q2.S, R12.2, R7.1, U$2.2, U$4.2, U$5.GNDA, U$5.GNDB, U$9.1, U2.AGND, U2.GND@3, U2.GND@5, U3.EXTINT, U3.GND6, U3.GND9, U5.GND, U6.GND, U7.VSS
- removed net MISO1: MISO.P, U$5.MISO, U2.PB4(MISO)
- removed net MOSI1: MOSI.P, U$5.MOSI, U2.PB3(MOSI/OC2)
- removed net N$11: R12.1, U7.PROG
- removed net N$12: C7.1, U2.AREF
- removed net N$13: !RES.P, C8.1, R5.1, U2.PC6(/RESET)
- removed net N$14: ANT.P, U$5.ANT
- removed net N$15: C12.1, Q1.2, U2.PB7(XTAL2/TOSC2)
- removed net N$16: C13.1, Q1.1, U2.PB6(XTAL1/TOSC1)
- removed net N$18: LED3.C, U7.STAT
- removed net N$19: Q2.G, R7.2, R8.1
- removed net N$2: R1.1, R9.2, U5.EN
- removed net N$20: R8.2, U2.PD6(AIN0)
- removed net N$21: Q2.D, R15.1, U$3.1
- removed net N$22: LED3.A, R13.2
- removed net N$24: C15.1, R13.1, U$4.1, U7.VIN
- removed net N$27: C4.1, C5.1, C6.1, R3.2, U3.+3V3, U5.VOUT
- removed net N$3: C18.1, C19.1, R2.1, R9.1, U5.VIN
- removed net N$7: LED1.A, R4.2
- removed net N$8: R4.1, U3.TM_GPIO5
- removed net N$9: U3.ON_OFF, U3.WAKEUP
- removed net RF_RTTY1: U$5.DIO2, U2.PC1(ADC1)
- removed net RXI1: R14.2, RXI_1.P, U2.PD0(RXD)
- removed net RXI_G1: R10.1, RXI1.P, U3.RXI
- removed net SCK1: SCK.P, U$5.SCK, U2.PB5(SCK)
- removed net TXO1: R10.2, TXO_.P, U2.PD1(TXD)
- removed net TXO_G1: R14.1, TXO1.P, U3.TXO
- new net BUZZER: R52.2, TP4.PP, U19.PB1(MISO)
- new net ENA: ENA.2, R51.2, U21.EN
- new net GND: BAT.2, C1.2, C2.2, C3.2, C4.2, C51.2, C52.2, C53.2, C54.2, C55.2, C58.2, CHAR.2, ENA.1, IC2.GND, LED10.C, LED11.C, Q10.S, R46.1, R53.2, U$17.1, U1.GND, U1.GND_2, U19.GND, U21.GND, U22.VSS, UART.1
- new net N$132: C53.1, R47.2, TP2.PP, U19.PB5(NRES)
- new net N$133: Q10.G, R45.2, R46.2, U$17.2
- new net N$134: LED10.A, R48.1
- new net N$137: LED11.A, R52.1
- new net N$138: PYRO.1, Q10.D
- new net N$139: R53.1, U22.PROG
- new net N$140: LED12.C, U22.STAT
- new net N$141: LED12.A, R54.2
- new net N$142: C58.1, CHAR.1, R54.1, U22.VIN
- new net N$5: C1.1, U1.CAP-A
- new net PYRO: R45.1, R48.2, U19.PB3(ADC3)
- new net SCL: IC2.SCL, R50.2, U1.SCL, U19.PB2(SCK/ADC1)
- new net SDA: IC2.SDA, R49.2, U1.SDA, U19.PB0(MOSI)
- new net UART: U19.PB4(ADC2), UART.2
- new net VBAT: BAT.1, C54.1, PYRO.2, R51.1, U21.VIN, U22.VBAT
- new net VCC: C3.1, C4.1, C51.1, C52.1, C55.1, IC2.VDD, R47.1, R49.1, R50.1, U1.VDD, U1.VDDIO, U19.VCC, U21.VOUT
- net N$6: now also C2.1, U1.CAP-R; no longer R3.1, U3.GPIO6
Other:
- moved on the sheet: C4
