File: eagle/gps_tracker_A2235h.brd (EAGLE design)
At the start: 62 x 28 mm, 53 parts, among them Q1 MC-405, U2 ATMEGA328P_TQFP, U3 A2235-H, U5 ADP160, U6 ADP160, U7 MCP73831

Commit message: Add files via upload
Parts:
- removed U$1: RFM69HW, hoperf:RFM
- added U$5: RFM69HW, gps_tracker:RFM
- moved C16 1.00 mm to (29.6, 3.84)
- moved C17 1.00 mm to (29.6, 2.57)
Connections:
- net !CS1: now also U$5.NSS; no longer U$1.NSS
- net !RF_RES1: now also U$5.RESET; no longer U$1.RESET
- net +3V3_1: now also U$5.VCC; no longer U$1.VCC
- net GND1: now also U$5.GNDA, U$5.GNDB; no longer U$1.GNDA, U$1.GNDB
- net MISO1: now also U$5.MISO; no longer U$1.MISO
- net MOSI1: now also U$5.MOSI; no longer U$1.MOSI
- net N$14: now also U$5.ANT; no longer U$1.ANT
- net RF_RTTY1: now also U$5.DIO2; no longer U$1.DIO2
- net SCK1: now also U$5.SCK; no longer U$1.SCK
Routing:
- net +3V3_1: track 65.2 -> 67.2 mm
- net GND1: vias 11 -> 13
- added copper zone on layer 16, net N$1
- added copper zone on layer 1, net N$4

Commit message: Add files via upload
Parts:
- added R15: 10k, rcl:R0603
- C10, C17, C19, C5, C7, C8: value (none) -> 100n
- C11, C6: value (none) -> 1n
- C12, C13: value (none) -> 22p
- C14, C15, C16, C18, C4, C9: value (none) -> 10uF
- R1, R10, R14, R2: value (none) -> 0
- R11, R3, R5: value (none) -> 10k
- R12: value (none) -> 2k7
- R13: value (none) -> 470
- R4, R8: value (none) -> 220
- R6, R7, R9: value (none) -> 100k
- moved U$3 1.50 mm to (2.54, 20.8)
Connections:
- net +3V3_1: now also R15.2
- net N$21: now also R15.1
Routing:
- net N$21: track 0.81 -> 4.17 mm
- net +3V3_1: track 67.2 -> 64.0 mm
- removed copper zone on layer 16, net N$1
- removed copper zone on layer 1, net N$4
Other:
- board text added: "1"
- board text added: "2"
- board text removed: "B"
- board text removed: "T"
