File: eagle/gps_tracker_org1411.brd (EAGLE design)
At the start: 62 x 28 mm, 59 parts, among them Q1 MC-405, Q3 200mA/50V, Q4 200mA/50V, U1 ORG1411, U2 ATMEGA328P_TQFP, U4 ADP160, U6 ADP160, U7 MCP73831

Commit message: Add files via upload
Parts:
- removed U$1: RFM69HW, hoperf:RFM
- added U$5: RFM69HW, gps_tracker:RFM
- moved C16 0.64 mm to (29.2, 3.84)
- moved C17 0.64 mm to (29.2, 2.57)
Connections:
- net !CS1: now also U$5.NSS; no longer U$1.NSS
- net !RF_RES1: now also U$5.RESET; no longer U$1.RESET
- net +3V3_1: now also U$5.VCC; no longer U$1.VCC
- net GND: now also U$5.GNDA, U$5.GNDB; no longer U$1.GNDA, U$1.GNDB
- net MISO1: now also U$5.MISO; no longer U$1.MISO
- net MOSI1: now also U$5.MOSI; no longer U$1.MOSI
- net N$14: now also U$5.ANT; no longer U$1.ANT
- net RF_RTTY1: now also U$5.DIO2; no longer U$1.DIO2
- net SCK1: now also U$5.SCK; no longer U$1.SCK
Routing:
- net N$14: track 2.59 -> 4.49 mm
- net +3V3_1: track 65.2 -> 66.4 mm
- net RF_RTTY1: track 21.6 -> 22.1 mm
- net GND: vias 12 -> 13
- added copper zone on layer 16, net N$7
- added copper zone on layer 1, net N$8

Commit message: Add files via upload
Parts:
- added R19: 10k, rcl:R0603
- C1, C14, C15, C16, C20, C9: value (none) -> 10uF
- C10, C17, C2, C21, C7, C8: value (none) -> 100n
- C11, C3: value (none) -> 1n
- C12, C13: value (none) -> 22p
- R1, R11, R5: value (none) -> 10k
- R10, R6, R7: value (none) -> 100k
- R12: value (none) -> 2k7
- R13: value (none) -> 470
- R14, R15, R16, R17: value (none) -> 2k2
- R18, R3, R4, R9: value (none) -> 0
- R2, R8: value (none) -> 220
- moved U$3 1.48 mm to (2.54, 20.8)
Connections:
- net +3V3_1: now also R19.2
- net N$21: now also R19.1
Routing:
- net N$21: track 0.81 -> 4.08 mm
- net +3V3_1: track 66.4 -> 65.1 mm
- removed copper zone on layer 16, net N$7
- removed copper zone on layer 1, net N$8
Other:
- board text added: "1"
- board text added: "2"
- board text removed: "B"
- board text removed: "T"
