File: eagle/gps_tracker_org1411.sch (EAGLE design)
At the start: 142 parts, among them IC2 MS563702BA03, Q1 MC-405, Q10 MOSFET-NCHANNELBSS123LT1G, Q13 MC-405, Q14 MOSFET-NCHANNELAO3404A, Q2 MOSFET-NCHANNELAO3404A, Q7 200mA/50V, Q8 200mA/50V, U10 ORG1411, U13 ADP160, U19 Tiny45-20-SMT, U2 ATMEGA328P_TQFP, U20 LIS3MDL, U21 ADP160, U22 MCP73831, U3 A2235-H, U34 ATMEGA328P_TQFP, U37 ADP160, U38 MCP73831, U5 ADP160, U6 ADP160, U7 MCP73831

Commit message: Add files via upload
Parts:
- removed !RES3, ANT2, MISO3, MOSI3, RXI1, RXI_1, RXI_5, SCK3, TXO1, TXO4, TXO_, TXO_3: (no value), wirepad:SMD2
- removed C101, C18, C19, C22, C23, C24, C4, C40, C41, C5, C53, C54, C55, C58, C6, C89, C90, C91, C92, C93, C94, C95, C96, C97, C98: (no value), rcl:C-EUC0603
- removed C51: 100nF, rcl:C-EUC0603
- removed C52: (no value), rcl:C-EUC1206
- removed C56: 0.22uF, rcl:C-EUC0603K
- removed C57: 0.22uF, rcl:C-EUC0603
- removed IC2: MS563702BA03, freetronics-original:MS563702BA03
- removed LED1, LED12, LED21, LED4: (no value), led:LEDCHIPLED_0603
- removed LED10, LED11: (no value), led:LEDCHIPLED_0805
- removed Q10: MOSFET-NCHANNELBSS123LT1G, SparkFun-DiscreteSemi:MOSFET-NCHANNELBSS123LT1G
- removed Q13: MC-405, gps_tracker:MC-405
- removed Q14: MOSFET-NCHANNELAO3404A, SparkFun-DiscreteSemi:MOSFET-NCHANNELAO3404A
- removed Q7, Q8: 200mA/50V, SparkFun-DiscreteSemi:MOSFET-NCHANNELBSS138
- removed R22, R23, R31, R35, R36, R45, R46, R47, R49, R50, R51, R53, R54, R88, R89, R90, R92, R93, R94, R95: (no value), rcl:R-EU_R0603
- removed R37, R38: (no value), rcl:R-EU_R1206
- removed R48, R52: 220, resistor:R-EU_R0603
- removed TP2, TP4: TPSB1,27, testpad:TPSB1,27
- removed U$14, U$15, U$16, U$17, U$18, U$36, U$37, U$38, U$39: 1X2, headers(2mm)(samtec):1X2
- removed U$35: RFM69HW, hoperf:RFM69HW
- removed U10: ORG1411, gps_tracker:ORG1411
- removed U13, U21, U37, U5: ADP160, SparkFun-PowerIC:ADP160
- removed U19: Tiny45-20-SMT, SparkFun-DigitalIC:ATTINY45TINY45-20-SMT
- removed U20: LIS3MDL, kg-ic:LIS3MDL
- removed U22, U38: MCP73831, SparkFun-PowerIC:MCP73831
- removed U3: A2235-H, gps_tracker:A2235-H
- removed U34: ATMEGA328P_TQFP, SparkFun-DigitalIC:ATMEGA328P_TQFP
- added C1, C2, C20, C21, C3: (no value), rcl:C-EUC0603
- added LED2: (no value), led:LEDCHIPLED_0603
- added Q3, Q4: 200mA/50V, SparkFun-DiscreteSemi:MOSFET-NCHANNELBSS138
- added R15, R18: (no value), rcl:R-EU_R0603
- added R16, R17: (no value), rcl:R-EU_R1206
- added RXI, TXO, TXOH: (no value), wirepad:SMD2
- added U1: ORG1411, gps_tracker:ORG1411
- added U4: ADP160, SparkFun-PowerIC:ADP160
Connections:
- removed net !CS2: R93.2, U$35.NSS, U34.PB1(OC1A)
- removed net !RF_RES2: U$35.RESET, U34.PD2(INT0)
- removed net +3V3_2: C91.1, C92.1, C93.1, C97.1, C98.1, R88.2, R93.1, U$35.VCC, U$37.2, U34.AVCC, U34.PC3(ADC3), U34.PD7(AIN1), U34.VCC@4, U34.VCC@6, U37.VOUT
- removed net +4.1V: R37.2, R38.2
- removed net +BAT1: C14.1, R2.2, R6.1, U$2.1, U6.VIN, U7.VBAT
- removed net +BAT2: C40.1, C41.1, C96.1, R31.1, R92.1, U$36.1, U13.VIN, U37.VIN, U38.VBAT
- removed net ANT2: ANT2.P, U$35.ANT
- removed net BUZZER: R52.2, TP4.PP, U19.PB1(MISO)
- removed net ENA1: R1.2, R6.2, U$9.2, U6.EN
- removed net ENA2: R31.2, R92.2, U$39.2, U13.EN, U37.EN
- removed net GND1: C10.2, C11.2, C12.2, C13.2, C14.2, C15.2, C16.2, C17.2, C18.2, C19.2, C4.2, C5.2, C6.2, C7.2, C8.2, C9.2, LED1.C, Q2.S, R12.2, R7.1, U$1.GNDA, U$1.GNDB, U$2.2, U$4.2, U$9.1, U2.AGND, U2.GND@3, U2.GND@5, U3.EXTINT, U3.GND6, U3.GND9, U5.GND, U6.GND, U7.VSS
- removed net GND2: C101.2, C22.2, C23.2, C24.2, C40.2, C41.2, C89.2, C90.2, C91.2, C92.2, C93.2, C94.2, C95.2, C96.2, C97.2, C98.2, LED4.C, Q14.S, R89.1, R94.2, U$35.GNDA, U$35.GNDB, U$36.2, U$38.2, U$39.1, U10.GND, U13.GND, U34.AGND, U34.GND@3, U34.GND@5, U37.GND, U38.VSS
- removed net MISO2: MISO3.P, U$35.MISO, U34.PB4(MISO)
- removed net MOSI2: MOSI3.P, U$35.MOSI, U34.PB3(MOSI/OC2)
- removed net N$132: C53.1, R47.2, TP2.PP, U19.PB5(NRES)
- removed net N$133: Q10.G, R45.2, R46.2, U$17.2
- removed net N$134: LED10.A, R48.1
- removed net N$135: C56.2, U20.C1
- removed net N$136: R51.2, U21.EN
- removed net N$137: LED11.A, R52.1
- removed net N$138: Q10.D, U$16.1
- removed net N$139: R53.1, U22.PROG
- removed net N$140: LED12.C, U22.STAT
- removed net N$141: LED12.A, R54.2
- removed net N$142: C58.1, R54.1, U$18.1, U22.VIN
- removed net N$162: C89.1, U34.AREF
- removed net N$163: !RES3.P, C90.1, R88.1, U34.PC6(/RESET)
- removed net N$165: C94.1, Q13.2, U34.PB7(XTAL2/TOSC2)
- removed net N$166: C95.1, Q13.1, U34.PB6(XTAL1/TOSC1)
- removed net N$167: Q14.G, R89.2, R90.1
- removed net N$168: R90.2, U34.PD6(AIN0)
- removed net N$169: Q14.D, U$37.1
- removed net N$171: R94.1, U38.PROG
- removed net N$172: LED21.C, U38.STAT
- removed net N$173: LED21.A, R95.2
- removed net N$174: C101.1, R95.1, U$38.1, U38.VIN
- removed net N$27: C4.1, C5.1, C6.1, R3.2, U3.+3V3, U5.VOUT
- removed net N$29: U10.ON/OFF, U10.WAKEUP
- removed net N$31: R23.1, U10.1PPS
- removed net N$54: Q7.S, R36.2, U10.TXO/MISO/SCL
- removed net N$55: Q7.D, R37.1, TXO4.P
- removed net N$56: Q8.D, R38.1, RXIH.P
- removed net N$57: Q8.S, R35.1, U10.RXI/MOSI/SDA
- removed net N$7: LED1.A, R4.2
- removed net N$8: R4.1, U3.TM_GPIO5
- removed net N$9: U3.ON_OFF, U3.WAKEUP
- removed net PYRO: R45.1, R48.2, U19.PB3(ADC3)
- removed net RF_RTTY2: U$35.DIO2, U34.PC1(ADC1)
- removed net RXI1: R14.2, RXI_1.P, U2.PD0(RXD)
- removed net RXI2: RXI_5.P, U34.PD0(RXD)
- removed net RXI_G1: R10.1, RXI1.P, U3.RXI
- removed net SCK2: SCK3.P, U$35.SCK, U34.PB5(SCK)
- removed net SCL: IC2.SCL, R50.2, U19.PB2(SCK/ADC1), U20.SCL/SPC
- removed net SDA: IC2.SDA, R49.2, U19.PB0(MOSI), U20.SDA/SDI
- removed net TXO1: R10.2, TXO_.P, U2.PD1(TXD)
- removed net TXO2: TXO_3.P, U34.PD1(TXD)
- removed net TXO_G1: R14.1, TXO1.P, U3.TXO
- removed net UART: U$15.2, U19.PB4(ADC2)
- removed net VBAT: C54.1, R51.1, U$14.1, U$16.2, U21.VIN, U22.VBAT
- removed net VCC: C51.1, C52.1, C55.1, C57.1, IC2.VDD, R47.1, R49.1, R50.1, U19.VCC, U20.CS, U20.SD0/SA1, U20.VDD, U20.VDD_IO, U21.VOUT
- new net +BAT: C14.1, R18.1, R6.1, U$2.1, U6.VIN, U7.VBAT
- new net ENA: R6.2, R9.2, U$9.2, U6.EN
- new net N$1: U1.ON/OFF, U1.WAKEUP
- new net N$26: Q3.D, R16.1, R3.2, TXOH.P
- new net N$4: LED2.A, R2.2
- new net N$5: Q3.S, R15.2, U1.TXO/MISO/SCL
- new net N1: R10.2, R9.1, U4.EN
- new net RXI: R3.1, RXI.P, U2.PD0(RXD)
- new net TXO: R4.1, TXO.P, U2.PD1(TXD)
- net GND: now also C1.2, C10.2, C11.2, C12.2, C13.2, C14.2, C15.2, C16.2, C17.2, C2.2, C20.2, C21.2, C3.2, C7.2, C8.2, C9.2, LED2.C, Q2.S, R12.2, R7.1, U$1.GNDA, U$1.GNDB, U$2.2, U$4.2, U$9.1, U1.GND, U2.AGND, U2.GND@3, U2.GND@5, U4.GND, U6.GND, U7.VSS; no longer C51.2, C52.2, C53.2, C54.2, C55.2, C56.1, C57.2, C58.2, IC2.GND, LED10.C, LED11.C, Q10.S, R46.1, R53.2, U$14.2, U$15.1, U$17.1, U$18.2, U19.GND, U20.GND, U20.RSVD1, U20.RSVD2, U21.GND, U22.VSS
- net N$2: now also U1.MODE1/SCK/!CTS; no longer R9.2, U5.EN
- net N$3: now also U1.1PPS; no longer C18.1, C19.1, R9.1, U5.VIN
- net N$30: now also Q4.D, R17.1, R4.2, RXIH.P; no longer R22.1, U10.MODE1/SCK/!CTS
- net N$32: now also Q4.S, R14.1, U1.RXI/MOSI/SDA; no longer LED4.A, R23.2
- net N$6: now also C20.1, C21.1, R10.1, R16.2, R17.2, R18.2, U4.VIN; no longer R3.1, U3.GPIO6
- net V+: now also C1.1, C2.1, C3.1, Q3.G, Q4.G, R1.2, R14.2, R15.1, U1.+1V8, U4.VOUT; no longer C22.1, C23.1, C24.1, Q7.G, Q8.G, R22.2, R35.2, R36.1, U10.+1V8, U13.VOUT

Commit message: Add files via upload
Parts:
- removed U$1: RFM69HW, hoperf:RFM69HW
- added U$5: RFM69HW, gps_tracker:RFM69HW
Connections:
- net !CS1: now also U$5.NSS; no longer U$1.NSS
- net !RF_RES1: now also U$5.RESET; no longer U$1.RESET
- net +3V3_1: now also U$5.VCC; no longer U$1.VCC
- net GND: now also U$5.GNDA, U$5.GNDB; no longer U$1.GNDA, U$1.GNDB
- net MISO1: now also U$5.MISO; no longer U$1.MISO
- net MOSI1: now also U$5.MOSI; no longer U$1.MOSI
- net N$14: now also U$5.ANT; no longer U$1.ANT
- net RF_RTTY1: now also U$5.DIO2; no longer U$1.DIO2
- net SCK1: now also U$5.SCK; no longer U$1.SCK

Commit message: Add files via upload
Parts:
- added R19: 10k, rcl:R-EU_R0603
- C1, C14, C15, C16, C20, C9: value (none) -> 10uF
- C10, C17, C2, C21, C7, C8: value (none) -> 100n
- C11, C3: value (none) -> 1n
- C12, C13: value (none) -> 22p
- R1, R11, R5: value (none) -> 10k
- R10, R6, R7: value (none) -> 100k
- R12: value (none) -> 2k7
- R13: value (none) -> 470
- R14, R15, R16, R17: value (none) -> 2k2
- R18, R3, R4, R9: value (none) -> 0
- R2, R8: value (none) -> 220
Connections:
- net +3V3_1: now also R19.2
- net N$21: now also R19.1
Changed lines of the file:
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@@
 <parts>
 <part name="GND3" library="supply1" deviceset="GND" device=""/>
-<part name="R1" library="rcl" deviceset="R-EU_" device="R0603"/>
-<part name="C1" library="rcl" deviceset="C-EU" device="C0603"/>
+<part name="R1" library="rcl" deviceset="R-EU_" device="R0603" value="10k"/>
+<part name="C1" library="rcl" deviceset="C-EU" device="C0603" value="10uF"/>
 <part name="LED2" library="led" deviceset="LED" device="CHIPLED_0603"/>
 <part name="U1" library="gps_tracker" deviceset="ORG1411" device=""/>
-<part name="R2" library="rcl" deviceset="R-EU_" device="R0603"/>
+<part name="R2" library="rcl" deviceset="R-EU_" device="R0603" value="220"/>
 <part name="GND5" library="supply1" deviceset="GND" device=""/>
 <part name="GND6" library="supply1" deviceset="GND" device=""/>
-<part name="C2" library="rcl" deviceset="C-EU" device="C0603"/>
+<part name="C2" library="rcl" deviceset="C-EU" device="C0603" value="100n"/>
 <part name="GND7" library="supply1" deviceset="GND" device=""/>
-<part name="C3" library="rcl" deviceset="C-EU" device="C0603"/>
+<part name="C3" library="rcl" deviceset="C-EU" device="C0603" value="1n"/>
 <part name="GND8" library="supply1" deviceset="GND" device=""/>
 <part name="U4" library="SparkFun-PowerIC" deviceset="ADP160" device="" value="ADP160">
@@
 </part>
 <part name="GND42" library="supply1" deviceset="GND" device=""/>
-<part name="C20" library="rcl" deviceset="C-EU" device="C0603"/>
+<part name="C20" library="rcl" deviceset="C-EU" device="C0603" value="10uF"/>
 <part name="GND43" library="supply1" deviceset="GND" device=""/>
-<part name="C21" library="rcl" deviceset="C-EU" device="C0603"/>
+<part name="C21" library="rcl" deviceset="C-EU" device="C0603" value="100n"/>
 <part name="GND44" library="supply1" deviceset="GND" device=""/>
-<part name="R10" library="rcl" deviceset="R-EU_" device="R0603"/>
+<part name="R10" library="rcl" deviceset="R-EU_" device="R0603" value="100k"/>
 <part name="P+1" library="supply1" deviceset="V+" device=""/>
-<part name="R14" library="rcl" deviceset="R-EU_" device="R0603"/>
-<part name="R15" library="rcl" deviceset="R-EU_" device="R0603"/>
-<part name="R16" library="rcl" deviceset="R-EU_" device="R1206"/>
+<part name="R14" library="rcl" deviceset="R-EU_" device="R0603" value="2k2"/>
+<part name="R15" library="rcl" deviceset="R-EU_" device="R0603" value="2k2"/>
+<part name="R16" library="rcl" deviceset="R-EU_" device="R1206" value="2k2"/>
 <part name="P+2" library="supply1" deviceset="V+" device=""/>
-<part name="R17" library="rcl" deviceset="R-EU_" device="R1206"/>
+<part name="R17" library="rcl" deviceset="R-EU_" device="R1206" value="2k2"/>
 <part name="TXOH" library="wirepad" deviceset="SMD2" device=""/>
 <part name="RXIH" library="wirepad" deviceset="SMD2" device=""/>
@@
 <part name="GND4" library="supply1" deviceset="GND" device=""/>
 <part name="+3V5" library="supply1" deviceset="+3V3" device=""/>
-<part name="C7" library="rcl" deviceset="C-EU" device="C0603"/>
+<part name="C7" library="rcl" deviceset="C-EU" device="C0603" value="100n"/>
 <part name="GND19" library="supply1" deviceset="GND" device=""/>
-<part name="C8" library="rcl" deviceset="C-EU" device="C0603"/>
+<part name="C8" library="rcl" deviceset="C-EU" device="C0603" value="100n"/>
 <part name="GND20" library="supply1" deviceset="GND" device=""/>
-<part name="R5" library="rcl" deviceset="R-EU_" device="R0603"/>
+<part name="R5" library="rcl" deviceset="R-EU_" device="R0603" value="10k"/>
 <part name="+3V10" library="supply1" deviceset="+3V3" device=""/>
-<part name="C9" library="rcl" deviceset="C-EU" device="C0603"/>
+<part name="C9" library="rcl" deviceset="C-EU" device="C0603" value="10uF"/>
 <part name="GND21" library="supply1" deviceset="GND" device=""/>
-<part name="C10" library="rcl" deviceset="C-EU" device="C0603"/>
+<part name="C10" library="rcl" deviceset="C-EU" device="C0603" value="100n"/>
 <part name="GND22" library="supply1" deviceset="GND" device=""/>
-<part name="C11" library="rcl" deviceset="C-EU" device="C0603"/>
+<part name="C11" library="rcl" deviceset="C-EU" device="C0603" value="1n"/>
 <part name="GND23" library="supply1" deviceset="GND" device=""/>
 <part name="+3V11" library="supply1" deviceset="+3V3" device=""/>
@@
 <part name="RXI" library="wirepad" deviceset="SMD2" device=""/>
 <part name="ANT" library="wirepad" deviceset="SMD2" device=""/>
-<part name="C12" library="rcl" deviceset="C-EU" device="C0603"/>
+<part name="C12" library="rcl" deviceset="C-EU" device="C0603" value="22p"/>
 <part name="GND26" library="supply1" deviceset="GND" device=""/>
-<part name="C13" library="rcl" deviceset="C-EU" device="C0603"/>
+<part name="C13" library="rcl" deviceset="C-EU" device="C0603" value="22p"/>
 <part name="GND27" library="supply1" deviceset="GND" device=""/>
 <part name="GND28" library="supply1" deviceset="GND" device=""/>
@@
 <attribute name="FARNELL" value="2508596"/>
 </part>
-<part name="C14" library="rcl" deviceset="C-EU" device="C0603"/>
+<part name="C14" library="rcl" deviceset="C-EU" device="C0603" value="10uF"/>
 <part name="GND29" library="supply1" deviceset="GND" device=""/>
 <part name="GND32" library="supply1" deviceset="GND" device=""/>
-<part name="C16" library="rcl" deviceset="C-EU" device="C0603"/>
+<part name="C16" library="rcl" deviceset="C-EU" device="C0603" value="10uF"/>
 <part name="GND33" library="supply1" deviceset="GND" device=""/>
-<part name="C17" library="rcl" deviceset="C-EU" device="C0603"/>
+<part name="C17" library="rcl" deviceset="C-EU" device="C0603" value="100n"/>
 <part name="GND34" library="supply1" deviceset="GND" device=""/>
 <part name="+3V16" library="supply1" deviceset="+3V3" device=""/>
@@
 <part name="Q2" library="SparkFun-DiscreteSemi" deviceset="MOSFET-NCHANNEL" device="AO3404A" value=""/>
 <part name="GND35" library="supply1" deviceset="GND" device=""/>
-<part name="R7" library="rcl" deviceset="R-EU_" device="R0603"/>
+<part name="R7" library="rcl" deviceset="R-EU_" device="R0603" value="100k"/>
 <part name="GND36" library="supply1" deviceset="GND" device=""/>
-<part name="R8" library="rcl" deviceset="R-EU_" device="R0603"/>
+<part name="R8" library="rcl" deviceset="R-EU_" device="R0603" value="220"/>
 <part name="U6" library="SparkFun-PowerIC" deviceset="ADP160" device="" value="ADP160">
 <attribute name="FARNELL" value="2510377 "/>
 </part>
-<part name="R6" library="rcl" deviceset="R-EU_" device="R0603"/>
+<part name="R6" library="rcl" deviceset="R-EU_" device="R0603" value="100k"/>
 <part name="U$2" library="headers(2mm)(samtec)" deviceset="1X2" device=""/>
-<part name="R11" library="rcl" deviceset="R-EU_" device="R0603"/>
+<part name="R11" library="rcl" deviceset="R-EU_" device="R0603" value="10k"/>
 <part name="+3V3" library="supply1" deviceset="+3V3" device=""/>
 <part name="+3V4" library="supply1" deviceset="+3V3" device=""/>
@@
 </part>
 <part name="GND9" library="supply1" deviceset="GND" device=""/>
-<part name="R12" library="rcl" deviceset="R-EU_" device="R0603"/>
+<part name="R12" library="rcl" deviceset="R-EU_" device="R0603" value="2k7"/>
 <part name="GND30" library="supply1" deviceset="GND" device=""/>
-<part name="R13" library="rcl" deviceset="R-EU_" device="R0603"/>
+<part name="R13" library="rcl" deviceset="R-EU_" device="R0603" value="470"/>
 <part name="LED3" library="led" deviceset="LED" device="CHIPLED_0603"/>
 <part name="U$4" library="headers(2mm)(samtec)" deviceset="1X2" device=""/>
 <part name="GND31" library="supply1" deviceset="GND" device=""/>
-<part name="C15" library="rcl" deviceset="C-EU" device="C0603"/>
+<part name="C15" library="rcl" deviceset="C-EU" device="C0603" value="10uF"/>
 <part name="GND45" library="supply1" deviceset="GND" device=""/>
 <part name="U$9" library="headers(2mm)(samtec)" deviceset="1X2" device=""/>
 <part name="GND15" library="supply1" deviceset="GND" device=""/>
-<part name="R3" library="rcl" deviceset="R-EU_" device="R0603"/>
-<part name="R4" library="rcl" deviceset="R-EU_" device="R0603"/>
-<part name="R9" library="rcl" deviceset="R-EU_" device="R0603"/>
-<part name="R18" library="rcl" deviceset="R-EU_" device="R0603"/>
+<part name="R3" library="rcl" deviceset="R-EU_" device="R0603" value="0"/>
+<part name="R4" library="rcl" deviceset="R-EU_" device="R0603" value="0"/>
+<part name="R9" library="rcl" deviceset="R-EU_" device="R0603" value="0"/>
+<part name="R18" library="rcl" deviceset="R-EU_" device="R0603" value="0"/>
 <part name="U$5" library="gps_tracker" deviceset="RFM69HW" device=""/>
+<part name="R19" library="rcl" deviceset="R-EU_" device="R0603" value="10k"/>
 </parts>
 <sheets>
@@
 <instance part="R18" gate="G$1" x="332.74" y="180.34"/>
 <instance part="U$5" gate="A" x="223.52" y="142.24"/>
+<instance part="R19" gate="G$1" x="276.86" y="91.44" rot="R90"/>
 </instances>
 <busses>
@@
 <pinref part="U$3" gate="G$1" pin="2"/>
 <wire x1="297.18" y1="93.98" x2="284.48" y2="93.98" width="0.1524" layer="91"/>
-<wire x1="284.48" y1="93.98" x2="284.48" y2="99.06" width="0.1524" layer="91"/>
+<wire x1="284.48" y1="93.98" x2="284.48" y2="96.52" width="0.1524" layer="91"/>
+<pinref part="R19" gate="G$1" pin="2"/>
+<wire x1="284.48" y1="96.52" x2="284.48" y2="99.06" width="0.1524" layer="91"/>
+<wire x1="276.86" y1="96.52" x2="284.48" y2="96.52" width="0.1524" layer="91"/>
+<junction x="284.48" y="96.52"/>
 </segment>
 </net>
@@
 <segment>
 <pinref part="Q2" gate="G$1" pin="D"/>
-<wire x1="284.48" y1="91.44" x2="284.48" y2="83.82" width="0.1524" layer="91"/>
+<wire x1="284.48" y1="91.44" x2="284.48" y2="86.36" width="0.1524" layer="91"/>
 <pinref part="U$3" gate="G$1" pin="1"/>
+<wire x1="284.48" y1="86.36" x2="284.48" y2="83.82" width="0.1524" layer="91"/>
 <wire x1="297.18" y1="91.44" x2="284.48" y2="91.44" width="0.1524" layer="91"/>
-</segment>
-</net>
+<pinref part="R19" gate="G$1" pin="1"/>
+<wire x1="276.86" y1="86.36" x2="284.48" y2="86.36" width="0.1524" layer="91"/>
+<junction x="284.48" y="86.36"/>
+</segment>
+</net>
